File: analogue_design/auto_cutoff_battery.kicad_pcb (KiCad board)
At the start: 2 copper layers, 100 x 52 mm, 56 parts, among them J1 RJ45, J2 RJ45, J3 Conn_01x01_Socket, J4 Conn_01x01_Socket, J5 Conn_01x03_Socket, J6 Conn_01x03_Socket, Q1 IRF540N, Q10 S8050, Q2 IRF9540N, Q3 S8050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

Commit message: finished V1
Parts:
- removed Bridge2: R, Resistor_THT:R_Axial_DIN0207_L6.3mm_D2.5mm_P5.08mm_Vertical
Routing:
- net BAT-: track 244.1 -> 260.3 mm
