File: analogue_design/auto_cutoff_battery.kicad_sch (KiCad schematic)
At the start: 56 parts, among them J1 RJ45, J2 RJ45, J3 Conn_01x01_Socket, J4 Conn_01x01_Socket, J5 Conn_01x03_Socket, J6 Conn_01x03_Socket, Q1 IRF540N, Q10 S8050, Q2 IRF9540N, Q3 S8050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

Commit message: finished V1
Parts:
- R15: value R -> 5k
- R16: value R -> 1.2k
Changed lines of the file:
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@@
       (effects (font (size 1.27 1.27)) (justify left))
     )
-    (property "Value" "R" (at -152.4 -24.13 0)
+    (property "Value" "1.2k" (at -152.4 -24.13 0)
       (effects (font (size 1.27 1.27)) (justify left))
     )
@@
       (effects (font (size 1.27 1.27)) (justify left))
     )
-    (property "Value" "R" (at -152.4 -31.75 0)
-      (effects (font (size 1.27 1.27)) (justify left))
-    )
+    (property "Value" "5k" (at -152.4 -31.75 0)
+      (effects (font (size 1.27 1.27)) (justify left))
+    )
