File: digital_design/Circuit/Circuit.kicad_sch (KiCad schematic)
At the start: 36 parts, among them J1 RJ45, J2 RJ45, J3 Conn_01x03_Socket, J4 Conn_01x03_Socket, J5 BAT+, J6 BAT-, Q1 IRF540N, Q2 IRF9540N, U1 PC817, U2 PC817, U3 LM7805_TO220, U4 PC817

Commit message: started updating
Parts:
- J3, J4: value Conn_01x03_Socket -> 01x03
Connections:
- net IN_OUT+: now also J3.2 (Pin_2); no longer J4.3 (Pin_3), Q2.3 (S)
- net BAT_OUT+: now reaches J4.1 (Pin_1)
- net BAT_OUT+: now also Q2.3 (S)
- removed net GNDD: C1.2, C2.2, D2.1 (K), D5.4 (K), Debug_pin1.1 (Pin_1), J6.1 (Pin_1), Q1.2 (D), R9.1, RV1.2, STC15W408AS_DIP16.8 (Pin_8), U1.2, U2.2, U3.2 (GND), U4.3
- removed net IN_OUT-: D2.2 (A), J3.1 (Pin_1), Q1.3 (S), U1.3, U2.3, U4.2
- new net: C1.2, Debug_pin1.1 (Pin_1), STC15W408AS_DIP16.8 (Pin_8)
- new net: D2.2 (A), U2.3
- new net: Q1.3 (S), U1.3
- new net: C2.2, U3.2 (GND)
- new net BAT-: U1.2, U2.2
- new net GND: J4.3 (Pin_3)
Other:
- moved on the sheet: J3, J4

Commit message: Updated Design as per requirement
Parts:
- removed D5: LED_BGRK, Connector_PinSocket_2.54mm:PinSocket_1x04_P2.54mm_Vertical, symbol Device:LED_BGRK
- removed RV1: 500ohm, Potentiometer_THT:Potentiometer_Bourns_3296W_Vertical, symbol Device:R_Potentiometer_Trim
- added D3: LED_BGKR, Connector_PinSocket_2.54mm:PinSocket_1x04_P2.54mm_Vertical, symbol Device:LED_BGKR
- added R6: 180, Resistor_THT:R_Axial_DIN0207_L6.3mm_D2.5mm_P7.62mm_Horizontal, symbol Device:R
- H1, H2, H3, H4: footprint MountingHole:MountingHole_5.3mm_M5_DIN965_Pad -> MountingHole:MountingHole_4mm
- J5, J6: footprint Connector_PinSocket_2.54mm:PinSocket_1x01_P2.54mm_Vertical -> MountingHole:MountingHole_3.2mm_M3_DIN965_Pad_TopBottom
- R11, R3: footprint Resistor_THT:R_Axial_DIN0207_L6.3mm_D2.5mm_P7.62mm_Horizontal -> Resistor_THT:R_Axial_DIN0207_L6.3mm_D2.5mm_P10.16mm_Horizontal
Connections:
- net BAT- is gone; now on net GNDD: U1.2, U2.2
- net GND is gone; now on net IN_OUT-: J4.3 (Pin_3)
- net IN_OUT+: now also R6.1
- net GNDD: now reaches C1.2, Debug_pin1.1 (Pin_1), STC15W408AS_DIP16.8 (Pin_8)
- net GNDD: now also C2.2, D2.1 (K), J6.1 (Pin_1), Q1.2 (D), R9.1, U3.2 (GND), U4.3, D3.3 (K)
- net at R12.2: now also D3.2 (GA)
- net at U4.1: now also R6.2
- net IN_OUT-: now reaches D2.2 (A), U2.3
- net IN_OUT-: now also Q1.3 (S), U1.3, U4.2
- net at R11.2: now also D3.1 (BA)
- net at R13.2: now also D3.4 (RA)

Commit message: changed holes footprint
Parts:
- H1, H2, H3, H4: footprint MountingHole:MountingHole_4mm -> MountingHole:MountingHole_4mm_Pad_TopBottom
Changed lines of the file:
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@@
       (effects (font (size 1.27 1.27)) (justify left))
     )
-    (property "Footprint" "MountingHole:MountingHole_4mm" (at 148.59 -152.4 0)
+    (property "Footprint" "MountingHole:MountingHole_4mm_Pad_TopBottom" (at 148.59 -152.4 0)
       (effects (font (size 1.27 1.27)) hide)
     )
@@
       (effects (font (size 1.27 1.27)) (justify left))
     )
-    (property "Footprint" "MountingHole:MountingHole_4mm" (at 148.348 -128.2044 0)
+    (property "Footprint" "MountingHole:MountingHole_4mm_Pad_TopBottom" (at 148.348 -128.2044 0)
       (effects (font (size 1.27 1.27)) hide)
     )
@@
       (effects (font (size 1.27 1.27)) (justify left))
     )
-    (property "Footprint" "MountingHole:MountingHole_4mm" (at 148.4766 -145.0535 0)
+    (property "Footprint" "MountingHole:MountingHole_4mm_Pad_TopBottom" (at 148.4766 -145.0535 0)
       (effects (font (size 1.27 1.27)) hide)
     )
@@
       (effects (font (size 1.27 1.27)) (justify left))
     )
-    (property "Footprint" "MountingHole:MountingHole_4mm" (at 148.4766 -136.5646 0)
-      (effects (font (size 1.27 1.27)) hide)
-    )
+    (property "Footprint" "MountingHole:MountingHole_4mm_Pad_TopBottom" (at 148.4766 -136.5646 0)
+      (effects (font (size 1.27 1.27)) hide)
+    )

Commit message: minor changes
Parts:
- R6: value 180 -> 1k
